File: pcb/Projekt_Schaltplan.kicad_sch (KiCad schematic)
At the start: 54 parts, among them J1 Conn_01x02_Pin, J10 Conn_01x02_Pin, J2 Conn_01x03_Pin, J3 Conn_01x05_Pin, J4 Conn_01x05_Pin, J5 Mini-DIN-6, J6 DA15_Socket, J7 Conn_01x02_Pin, J8 Conn_01x02_Pin, J9 Conn_01x02_Pin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

Commit message: [refactoring, feat] adding documentation and refactoring pcb annotation
Other:
- note added: "Mounting Holes and Miscellaneous"
- note removed: "Mounting Holes and Miscelleanious"
Changed lines of the file:
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@@
 		)
 	)
-	(text "Mounting Holes and Miscelleanious"
+	(text "Mounting Holes and Miscellaneous"
 		(exclude_from_sim no)
 		(at 378.968 249.936 0)
